Commit message: fix: corrigir referências de pacotes e setup.py para arquitectura de pacote único
- launch files: substituir get_package_share_directory('yahboomcar_*') por
  caminhos relativos ao share do robodog2 (pacotes yahboomcar_* não são
  registados separadamente pelo colcon por estarem dentro de robodog2/)
- urdf/rbd_X3_sim.urdf.xacro: meshes package://yahboomcar_description →
  package://robodog2/yahboomcar_description (necessário para Gazebo resolver)
- setup.py: adicionar data_files para yahboomcar_bringup/param, rviz,
  yahboomcar_description/meshes (mecanum, Ackermann, sensor),
  yahboomcar_nav/launch, params, rviz, maps, yahboomcar_laser/launch
- rbd_slam_toolbox_params.yaml: min_laser_range 0.0 → 0.1 (warning SLAM)

Problema identificado: pacotes yahboomcar_* aninhados dentro de robodog2/
causam conflito de identidade — colcon só vê robodog2. Próximo passo:
estudar a estrutura real do Rosmaster X3 para decidir arquitectura correcta.

Co-Authored-By: Claude Sonnet 4.6 <noreply@anthropic.com>

File: urdf/rbd_X3_sim.urdf.xacro (robot description, xacro)
@@ -42,5 +42,5 @@
       <origin xyz="0 0 0" rpy="0 0 0"/>
       <geometry>
-        <mesh filename="package://yahboomcar_description/meshes/mecanum/base_link_X3.STL"/>
+        <mesh filename="package://robodog2/yahboomcar_description/meshes/mecanum/base_link_X3.STL"/>
       </geometry>
       <material name="Green"><color rgba="0 0.7 0 1"/></material>
@@ -49,5 +49,5 @@
       <origin xyz="0 0 0" rpy="0 0 0"/>
       <geometry>
-        <mesh filename="package://yahboomcar_description/meshes/mecanum/base_link_X3.STL"/>
+        <mesh filename="package://robodog2/yahboomcar_description/meshes/mecanum/base_link_X3.STL"/>
       </geometry>
     </collision>
@@ -74,5 +74,5 @@
       <origin xyz="0 0 0" rpy="0 0 0"/>
       <geometry>
-        <mesh filename="package://yahboomcar_description/meshes/mecanum/front_right_wheel_X3.STL"/>
+        <mesh filename="package://robodog2/yahboomcar_description/meshes/mecanum/front_right_wheel_X3.STL"/>
       </geometry>
       <material name="LightGray"><color rgba="0.7 0.7 0.7 1"/></material>
@@ -81,5 +81,5 @@
       <origin xyz="0 0 0" rpy="0 0 0"/>
       <geometry>
-        <mesh filename="package://yahboomcar_description/meshes/mecanum/front_right_wheel_X3.STL"/>
+        <mesh filename="package://robodog2/yahboomcar_description/meshes/mecanum/front_right_wheel_X3.STL"/>
       </geometry>
     </collision>
@@ -103,12 +103,12 @@
       <origin xyz="0 0 0" rpy="0 0 0"/>
       <geometry>
-        <mesh filename="package://yahboomcar_description/meshes/mecanum/front_left_wheel_X3.STL"/>
-      </geometry>
-      <material name="LightGray"/>
-    </visual>
-    <collision>
-      <origin xyz="0 0 0" rpy="0 0 0"/>
-      <geometry>
-        <mesh filename="package://yahboomcar_description/meshes/mecanum/front_left_wheel_X3.STL"/>
+        <mesh filename="package://robodog2/yahboomcar_description/meshes/mecanum/front_left_wheel_X3.STL"/>
+      </geometry>
+      <material name="LightGray"/>
+    </visual>
+    <collision>
+      <origin xyz="0 0 0" rpy="0 0 0"/>
+      <geometry>
+        <mesh filename="package://robodog2/yahboomcar_description/meshes/mecanum/front_left_wheel_X3.STL"/>
       </geometry>
     </collision>
@@ -132,12 +132,12 @@
       <origin xyz="0 0 0" rpy="0 0 0"/>
       <geometry>
-        <mesh filename="package://yahboomcar_description/meshes/mecanum/back_right_wheel_X3.STL"/>
-      </geometry>
-      <material name="LightGray"/>
-    </visual>
-    <collision>
-      <origin xyz="0 0 0" rpy="0 0 0"/>
-      <geometry>
-        <mesh filename="package://yahboomcar_description/meshes/mecanum/back_right_wheel_X3.STL"/>
+        <mesh filename="package://robodog2/yahboomcar_description/meshes/mecanum/back_right_wheel_X3.STL"/>
+      </geometry>
+      <material name="LightGray"/>
+    </visual>
+    <collision>
+      <origin xyz="0 0 0" rpy="0 0 0"/>
+      <geometry>
+        <mesh filename="package://robodog2/yahboomcar_description/meshes/mecanum/back_right_wheel_X3.STL"/>
       </geometry>
     </collision>
@@ -161,12 +161,12 @@
       <origin xyz="0 0 0" rpy="0 0 0"/>
       <geometry>
-        <mesh filename="package://yahboomcar_description/meshes/mecanum/back_left_wheel_X3.STL"/>
-      </geometry>
-      <material name="LightGray"/>
-    </visual>
-    <collision>
-      <origin xyz="0 0 0" rpy="0 0 0"/>
-      <geometry>
-        <mesh filename="package://yahboomcar_description/meshes/mecanum/back_left_wheel_X3.STL"/>
+        <mesh filename="package://robodog2/yahboomcar_description/meshes/mecanum/back_left_wheel_X3.STL"/>
+      </geometry>
+      <material name="LightGray"/>
+    </visual>
+    <collision>
+      <origin xyz="0 0 0" rpy="0 0 0"/>
+      <geometry>
+        <mesh filename="package://robodog2/yahboomcar_description/meshes/mecanum/back_left_wheel_X3.STL"/>
       </geometry>
     </collision>
@@ -190,12 +190,12 @@
       <origin xyz="0 0 0" rpy="0 0 0"/>
       <geometry>
-        <mesh filename="package://yahboomcar_description/meshes/sensor/laser_link.STL"/>
-      </geometry>
-      <material name="LightGray"/>
-    </visual>
-    <collision>
-      <origin xyz="0 0 0" rpy="0 0 0"/>
-      <geometry>
-        <mesh filename="package://yahboomcar_description/meshes/sensor/laser_link.STL"/>
+        <mesh filename="package://robodog2/yahboomcar_description/meshes/sensor/laser_link.STL"/>
+      </geometry>
+      <material name="LightGray"/>
+    </visual>
+    <collision>
+      <origin xyz="0 0 0" rpy="0 0 0"/>
+      <geometry>
+        <mesh filename="package://robodog2/yahboomcar_description/meshes/sensor/laser_link.STL"/>
       </geometry>
     </collision>
@@ -216,12 +216,12 @@
       <origin xyz="0 0 0" rpy="0 0 0"/>
       <geometry>
-        <mesh filename="package://yahboomcar_description/meshes/sensor/camera_link.STL"/>
-      </geometry>
-      <material name="LightGray"/>
-    </visual>
-    <collision>
-      <origin xyz="0 0 0" rpy="0 0 0"/>
-      <geometry>
-        <mesh filename="package://yahboomcar_description/meshes/sensor/camera_link.STL"/>
+        <mesh filename="package://robodog2/yahboomcar_description/meshes/sensor/camera_link.STL"/>
+      </geometry>
+      <material name="LightGray"/>
+    </visual>
+    <collision>
+      <origin xyz="0 0 0" rpy="0 0 0"/>
+      <geometry>
+        <mesh filename="package://robodog2/yahboomcar_description/meshes/sensor/camera_link.STL"/>
       </geometry>
     </collision>

Commit message: refactor: mover yahboomcar_* para pacotes irmãos em ros2_ws/src/
Os pacotes yahboomcar_bringup/description/laser/nav eram subpastas dentro
de robodog2, impedindo o colcon de os registar como pacotes independentes.
Movidos para ~/ros2_ws/src/ como irmãos de robodog2.

Consequências:
- package://yahboomcar_description/meshes/... resolve no Gazebo (robô visível)
- get_package_share_directory('yahboomcar_nav') funciona sem workaround
- setup.py limpo (removidas entradas data_files das subpastas)
- launch files revertidos para caminhos directos via get_package_share_directory

Co-Authored-By: Claude Sonnet 4.6 <noreply@anthropic.com>

File: urdf/rbd_X3_sim.urdf.xacro (robot description, xacro)
@@ -42,5 +42,5 @@
       <origin xyz="0 0 0" rpy="0 0 0"/>
       <geometry>
-        <mesh filename="package://robodog2/yahboomcar_description/meshes/mecanum/base_link_X3.STL"/>
+        <mesh filename="package://yahboomcar_description/meshes/mecanum/base_link_X3.STL"/>
       </geometry>
       <material name="Green"><color rgba="0 0.7 0 1"/></material>
@@ -49,5 +49,5 @@
       <origin xyz="0 0 0" rpy="0 0 0"/>
       <geometry>
-        <mesh filename="package://robodog2/yahboomcar_description/meshes/mecanum/base_link_X3.STL"/>
+        <mesh filename="package://yahboomcar_description/meshes/mecanum/base_link_X3.STL"/>
       </geometry>
     </collision>
@@ -74,5 +74,5 @@
       <origin xyz="0 0 0" rpy="0 0 0"/>
       <geometry>
-        <mesh filename="package://robodog2/yahboomcar_description/meshes/mecanum/front_right_wheel_X3.STL"/>
+        <mesh filename="package://yahboomcar_description/meshes/mecanum/front_right_wheel_X3.STL"/>
       </geometry>
       <material name="LightGray"><color rgba="0.7 0.7 0.7 1"/></material>
@@ -81,5 +81,5 @@
       <origin xyz="0 0 0" rpy="0 0 0"/>
       <geometry>
-        <mesh filename="package://robodog2/yahboomcar_description/meshes/mecanum/front_right_wheel_X3.STL"/>
+        <mesh filename="package://yahboomcar_description/meshes/mecanum/front_right_wheel_X3.STL"/>
       </geometry>
     </collision>
@@ -103,12 +103,12 @@
       <origin xyz="0 0 0" rpy="0 0 0"/>
       <geometry>
-        <mesh filename="package://robodog2/yahboomcar_description/meshes/mecanum/front_left_wheel_X3.STL"/>
-      </geometry>
-      <material name="LightGray"/>
-    </visual>
-    <collision>
-      <origin xyz="0 0 0" rpy="0 0 0"/>
-      <geometry>
-        <mesh filename="package://robodog2/yahboomcar_description/meshes/mecanum/front_left_wheel_X3.STL"/>
+        <mesh filename="package://yahboomcar_description/meshes/mecanum/front_left_wheel_X3.STL"/>
+      </geometry>
+      <material name="LightGray"/>
+    </visual>
+    <collision>
+      <origin xyz="0 0 0" rpy="0 0 0"/>
+      <geometry>
+        <mesh filename="package://yahboomcar_description/meshes/mecanum/front_left_wheel_X3.STL"/>
       </geometry>
     </collision>
@@ -132,12 +132,12 @@
       <origin xyz="0 0 0" rpy="0 0 0"/>
       <geometry>
-        <mesh filename="package://robodog2/yahboomcar_description/meshes/mecanum/back_right_wheel_X3.STL"/>
-      </geometry>
-      <material name="LightGray"/>
-    </visual>
-    <collision>
-      <origin xyz="0 0 0" rpy="0 0 0"/>
-      <geometry>
-        <mesh filename="package://robodog2/yahboomcar_description/meshes/mecanum/back_right_wheel_X3.STL"/>
+        <mesh filename="package://yahboomcar_description/meshes/mecanum/back_right_wheel_X3.STL"/>
+      </geometry>
+      <material name="LightGray"/>
+    </visual>
+    <collision>
+      <origin xyz="0 0 0" rpy="0 0 0"/>
+      <geometry>
+        <mesh filename="package://yahboomcar_description/meshes/mecanum/back_right_wheel_X3.STL"/>
       </geometry>
     </collision>
@@ -161,12 +161,12 @@
       <origin xyz="0 0 0" rpy="0 0 0"/>
       <geometry>
-        <mesh filename="package://robodog2/yahboomcar_description/meshes/mecanum/back_left_wheel_X3.STL"/>
-      </geometry>
-      <material name="LightGray"/>
-    </visual>
-    <collision>
-      <origin xyz="0 0 0" rpy="0 0 0"/>
-      <geometry>
-        <mesh filename="package://robodog2/yahboomcar_description/meshes/mecanum/back_left_wheel_X3.STL"/>
+        <mesh filename="package://yahboomcar_description/meshes/mecanum/back_left_wheel_X3.STL"/>
+      </geometry>
+      <material name="LightGray"/>
+    </visual>
+    <collision>
+      <origin xyz="0 0 0" rpy="0 0 0"/>
+      <geometry>
+        <mesh filename="package://yahboomcar_description/meshes/mecanum/back_left_wheel_X3.STL"/>
       </geometry>
     </collision>
@@ -190,12 +190,12 @@
       <origin xyz="0 0 0" rpy="0 0 0"/>
       <geometry>
-        <mesh filename="package://robodog2/yahboomcar_description/meshes/sensor/laser_link.STL"/>
-      </geometry>
-      <material name="LightGray"/>
-    </visual>
-    <collision>
-      <origin xyz="0 0 0" rpy="0 0 0"/>
-      <geometry>
-        <mesh filename="package://robodog2/yahboomcar_description/meshes/sensor/laser_link.STL"/>
+        <mesh filename="package://yahboomcar_description/meshes/sensor/laser_link.STL"/>
+      </geometry>
+      <material name="LightGray"/>
+    </visual>
+    <collision>
+      <origin xyz="0 0 0" rpy="0 0 0"/>
+      <geometry>
+        <mesh filename="package://yahboomcar_description/meshes/sensor/laser_link.STL"/>
       </geometry>
     </collision>
@@ -216,12 +216,12 @@
       <origin xyz="0 0 0" rpy="0 0 0"/>
       <geometry>
-        <mesh filename="package://robodog2/yahboomcar_description/meshes/sensor/camera_link.STL"/>
-      </geometry>
-      <material name="LightGray"/>
-    </visual>
-    <collision>
-      <origin xyz="0 0 0" rpy="0 0 0"/>
-      <geometry>
-        <mesh filename="package://robodog2/yahboomcar_description/meshes/sensor/camera_link.STL"/>
+        <mesh filename="package://yahboomcar_description/meshes/sensor/camera_link.STL"/>
+      </geometry>
+      <material name="LightGray"/>
+    </visual>
+    <collision>
+      <origin xyz="0 0 0" rpy="0 0 0"/>
+      <geometry>
+        <mesh filename="package://yahboomcar_description/meshes/sensor/camera_link.STL"/>
       </geometry>
     </collision>

Commit message: fix: corrigir spawn do robot em Gazebo e geometria de colisão URDF
- rbd_casa_x3_launch.py: reescrito como auto-suficiente (padrão robodog1)
  Gazebo arranca pausado (pause:=true) para evitar deslocamento do robot
  durante o carregamento dos 178 modelos do cma_moveis.world;
  RegisterEventHandler(OnProcessExit) chama /unpause_physics após spawn.

- rbd_sim_minimal_launch.py: novo launch de diagnóstico com empty.world
  sem imu_filter_madgwick, para verificar pipeline Gazebo de forma isolada.

- rbd_X3_sim.urdf.xacro: colisões STL substituídas por formas simples
  O motor ODE não detectava contacto entre as malhas STL e o ground plane,
  fazendo o robot cair indefinidamente (z=-50m). Fix: box para base_link,
  cilindros para rodas/laser, box para camera_link + massa mínima 0.01kg.
  Resultado: /odom z≈-0.009m (robot na superfície). Visuais STL mantidos.

Co-Authored-By: Claude Sonnet 4.6 <noreply@anthropic.com>

File: urdf/rbd_X3_sim.urdf.xacro (robot description, xacro)
@@ -49,5 +49,5 @@
       <origin xyz="0 0 0" rpy="0 0 0"/>
       <geometry>
-        <mesh filename="package://yahboomcar_description/meshes/mecanum/base_link_X3.STL"/>
+        <box size="0.25 0.20 0.08"/>
       </geometry>
     </collision>
@@ -81,5 +81,5 @@
       <origin xyz="0 0 0" rpy="0 0 0"/>
       <geometry>
-        <mesh filename="package://yahboomcar_description/meshes/mecanum/front_right_wheel_X3.STL"/>
+        <cylinder radius="0.033" length="0.028"/>
       </geometry>
     </collision>
@@ -110,5 +110,5 @@
       <origin xyz="0 0 0" rpy="0 0 0"/>
       <geometry>
-        <mesh filename="package://yahboomcar_description/meshes/mecanum/front_left_wheel_X3.STL"/>
+        <cylinder radius="0.033" length="0.028"/>
       </geometry>
     </collision>
@@ -139,5 +139,5 @@
       <origin xyz="0 0 0" rpy="0 0 0"/>
       <geometry>
-        <mesh filename="package://yahboomcar_description/meshes/mecanum/back_right_wheel_X3.STL"/>
+        <cylinder radius="0.033" length="0.028"/>
       </geometry>
     </collision>
@@ -168,5 +168,5 @@
       <origin xyz="0 0 0" rpy="0 0 0"/>
       <geometry>
-        <mesh filename="package://yahboomcar_description/meshes/mecanum/back_left_wheel_X3.STL"/>
+        <cylinder radius="0.033" length="0.028"/>
       </geometry>
     </collision>
@@ -197,5 +197,5 @@
       <origin xyz="0 0 0" rpy="0 0 0"/>
       <geometry>
-        <mesh filename="package://yahboomcar_description/meshes/sensor/laser_link.STL"/>
+        <cylinder radius="0.025" length="0.035"/>
       </geometry>
     </collision>
@@ -210,6 +210,6 @@
     <inertial>
       <origin xyz="0 0 0" rpy="0 0 0"/>
-      <mass value="0"/>
-      <inertia ixx="0" ixy="0" ixz="0" iyy="0" iyz="0" izz="0"/>
+      <mass value="0.01"/>
+      <inertia ixx="1e-6" ixy="0" ixz="0" iyy="1e-6" iyz="0" izz="1e-6"/>
     </inertial>
     <visual>
@@ -223,5 +223,5 @@
       <origin xyz="0 0 0" rpy="0 0 0"/>
       <geometry>
-        <mesh filename="package://yahboomcar_description/meshes/sensor/camera_link.STL"/>
+        <box size="0.025 0.050 0.020"/>
       </geometry>
     </collision>

Commit message: feat: adicionar meshes STL ao robodog2 e corrigir referências de pacote no URDF
- Copiada pasta meshes/ (mecanum + sensor STLs) do rosmaster_x3 para dentro do pacote robodog2
- Corrigidas todas as referências package://yahboomcar_description/meshes/ → package://robodog2/meshes/ em rbd_X3_sim.urdf.xacro
- Adicionadas entradas meshes/mecanum e meshes/sensor ao setup.py para instalação correcta via colcon

Co-Authored-By: Claude Sonnet 4.6 <noreply@anthropic.com>

File: urdf/rbd_X3_sim.urdf.xacro (robot description, xacro)
@@ -5,5 +5,5 @@
   Adaptado de yahboomcar_X3_sim.urdf.xacro (ROS1/robodog1).
   Alterações em relação ao original ROS1:
-    1. Caminhos das malhas: package://robodog1 → package://yahboomcar_description
+    1. Caminhos das malhas: package://robodog1 → package://robodog2
        Sufixo _X3 adicionado nos ficheiros da pasta mecanum/ (ex: base_link_X3.STL).
     2. Plugin planar_move: parâmetros renomeados para convenção ROS2 (snake_case).
@@ -42,5 +42,5 @@
       <origin xyz="0 0 0" rpy="0 0 0"/>
       <geometry>
-        <mesh filename="package://yahboomcar_description/meshes/mecanum/base_link_X3.STL"/>
+        <mesh filename="package://robodog2/meshes/mecanum/base_link_X3.STL"/>
       </geometry>
       <material name="Green"><color rgba="0 0.7 0 1"/></material>
@@ -74,5 +74,5 @@
       <origin xyz="0 0 0" rpy="0 0 0"/>
       <geometry>
-        <mesh filename="package://yahboomcar_description/meshes/mecanum/front_right_wheel_X3.STL"/>
+        <mesh filename="package://robodog2/meshes/mecanum/front_right_wheel_X3.STL"/>
       </geometry>
       <material name="LightGray"><color rgba="0.7 0.7 0.7 1"/></material>
@@ -103,5 +103,5 @@
       <origin xyz="0 0 0" rpy="0 0 0"/>
       <geometry>
-        <mesh filename="package://yahboomcar_description/meshes/mecanum/front_left_wheel_X3.STL"/>
+        <mesh filename="package://robodog2/meshes/mecanum/front_left_wheel_X3.STL"/>
       </geometry>
       <material name="LightGray"/>
@@ -132,5 +132,5 @@
       <origin xyz="0 0 0" rpy="0 0 0"/>
       <geometry>
-        <mesh filename="package://yahboomcar_description/meshes/mecanum/back_right_wheel_X3.STL"/>
+        <mesh filename="package://robodog2/meshes/mecanum/back_right_wheel_X3.STL"/>
       </geometry>
       <material name="LightGray"/>
@@ -161,5 +161,5 @@
       <origin xyz="0 0 0" rpy="0 0 0"/>
       <geometry>
-        <mesh filename="package://yahboomcar_description/meshes/mecanum/back_left_wheel_X3.STL"/>
+        <mesh filename="package://robodog2/meshes/mecanum/back_left_wheel_X3.STL"/>
       </geometry>
       <material name="LightGray"/>
@@ -190,5 +190,5 @@
       <origin xyz="0 0 0" rpy="0 0 0"/>
       <geometry>
-        <mesh filename="package://yahboomcar_description/meshes/sensor/laser_link.STL"/>
+        <mesh filename="package://robodog2/meshes/sensor/laser_link.STL"/>
       </geometry>
       <material name="LightGray"/>
@@ -216,5 +216,5 @@
       <origin xyz="0 0 0" rpy="0 0 0"/>
       <geometry>
-        <mesh filename="package://yahboomcar_description/meshes/sensor/camera_link.STL"/>
+        <mesh filename="package://robodog2/meshes/sensor/camera_link.STL"/>
       </geometry>
       <material name="LightGray"/>

Commit message: fix: corrigir movimento mecanum — fricção anisotrópica nas rodas
Sem parâmetros de atrito ODE, o motor de física tratava as rodas como
cilindros isotrópicos: só gerava força longitudinal, impedindo rotação
e movimento lateral.

Alterações:
- Colisão de cada roda: cilindro → esfera (raio=0.033 m), necessário
  para contacto limpo com o modelo de fricção ODE
- Adicionados mu=1.0, mu2=0.0 e fdir1 por roda:
    FL: [1,0,-1]  FR: [-1,0,-1]
    BL: [1,0,1]   BR: [-1,0,1]
  (fdir1 calculado no frame do link a partir da diagonal do chassi,
   seguindo o exemplo oficial gz-sim8/worlds/mecanum_drive.sdf)

Co-Authored-By: Claude Sonnet 4.6 <noreply@anthropic.com>

File: urdf/rbd_X3_sim.urdf.xacro (robot description, xacro)
@@ -81,5 +81,5 @@
       <origin xyz="0 0 0" rpy="0 0 0"/>
       <geometry>
-        <cylinder radius="0.033" length="0.028"/>
+        <sphere radius="0.033"/>
       </geometry>
     </collision>
@@ -110,5 +110,5 @@
       <origin xyz="0 0 0" rpy="0 0 0"/>
       <geometry>
-        <cylinder radius="0.033" length="0.028"/>
+        <sphere radius="0.033"/>
       </geometry>
     </collision>
@@ -139,5 +139,5 @@
       <origin xyz="0 0 0" rpy="0 0 0"/>
       <geometry>
-        <cylinder radius="0.033" length="0.028"/>
+        <sphere radius="0.033"/>
       </geometry>
     </collision>
@@ -168,5 +168,5 @@
       <origin xyz="0 0 0" rpy="0 0 0"/>
       <geometry>
-        <cylinder radius="0.033" length="0.028"/>
+        <sphere radius="0.033"/>
       </geometry>
     </collision>
@@ -237,8 +237,33 @@
   <!-- Cores Gazebo -->
   <gazebo reference="base_link"><material>Gazebo/Green</material></gazebo>
-  <gazebo reference="front_right_wheel"><material>Gazebo/DarkGrey</material></gazebo>
-  <gazebo reference="front_left_wheel"><material>Gazebo/DarkGrey</material></gazebo>
-  <gazebo reference="back_right_wheel"><material>Gazebo/DarkGrey</material></gazebo>
-  <gazebo reference="back_left_wheel"><material>Gazebo/DarkGrey</material></gazebo>
+  <!-- Fricção anisotrópica para simulação de rodas mecanum.
+       mu=1.0 na direção de tração (fdir1), mu2=0.0 na direção livre do rolo.
+       fdir1 calculado no frame do link a partir da diagonal no frame do chassi:
+         FL/BL chassis [1,±1,0] → link Rx(+π/2)  → FL:[1,0,-1]  BL:[1,0,1]
+         FR/BR chassis [1,±1,0] → link Rz(π)Rx(-π/2) → FR:[-1,0,-1] BR:[-1,0,1] -->
+  <gazebo reference="front_right_wheel">
+    <material>Gazebo/DarkGrey</material>
+    <mu>1.0</mu>
+    <mu2>0.0</mu2>
+    <fdir1>-1 0 -1</fdir1>
+  </gazebo>
+  <gazebo reference="front_left_wheel">
+    <material>Gazebo/DarkGrey</material>
+    <mu>1.0</mu>
+    <mu2>0.0</mu2>
+    <fdir1>1 0 -1</fdir1>
+  </gazebo>
+  <gazebo reference="back_right_wheel">
+    <material>Gazebo/DarkGrey</material>
+    <mu>1.0</mu>
+    <mu2>0.0</mu2>
+    <fdir1>-1 0 1</fdir1>
+  </gazebo>
+  <gazebo reference="back_left_wheel">
+    <material>Gazebo/DarkGrey</material>
+    <mu>1.0</mu>
+    <mu2>0.0</mu2>
+    <fdir1>1 0 1</fdir1>
+  </gazebo>
   <gazebo reference="laser_link"><material>Gazebo/FlatBlack</material></gazebo>
   <!--
