Commit message: fix: corrigir eixo de rotação das rodas direitas (FR/BR) para MecanumDrive
As rodas direitas têm rpy="-π/2, 0, π" → eixo Z_link aponta em -Y_world.
Com axis="0 0 1", velocidade positiva = rolar para trás nessas rodas,
o oposto das esquerdas. O plugin MecanumDrive assume que velocidade
positiva = frente para todas as rodas → inversão + rotação instável.

Correcção: axis="0 0 -1" para front_right_joint e back_right_joint.
Com axis="0 0 -1", positivo → rotação em -Z_link = +Y_world → frente,
consistente com as rodas esquerdas (axis="0 0 1", Z_link = +Y_world).

As rodas esquerdas (rpy="+π/2, 0, 0", Z_link = +Y_world) ficam inalteradas.
Os valores de fdir1 não mudam pois são no frame do link (definido pelo RPY,
não pelo axis).

Co-Authored-By: Claude Sonnet 4.6 <noreply@anthropic.com>

File: urdf/rbd_X3_sim.urdf.xacro (robot description, xacro)
@@ -89,5 +89,5 @@
     <parent link="base_link"/>
     <child link="front_right_wheel"/>
-    <axis xyz="0 0 1" rpy="0 0 0"/>
+    <axis xyz="0 0 -1" rpy="0 0 0"/>
     <limit effort="100" velocity="1"/>
   </joint>
@@ -147,5 +147,5 @@
     <parent link="base_link"/>
     <child link="back_right_wheel"/>
-    <axis xyz="0 0 1" rpy="0 0 0"/>
+    <axis xyz="0 0 -1" rpy="0 0 0"/>
     <limit effort="100" velocity="1"/>
   </joint>
